File: kicad/MAPusart.kicad_pcb (KiCad board)
At the start: 2 copper layers, 15 x 19 mm, 9 parts, among them J3 USB-Micro, U3 CP210X

Commit message: MAPusart schematic, PCB complete. Bom pending
Parts:
- added D1: USBLC6-2, MAPusart.pretty:SOT-23-6, B.Cu at (114.7, 35.0)
- Z3: footprint MAPone.pretty:MA_Logo2 -> MAPusart.pretty:MA_Logo2
- Z5: footprint MAPone:OSHW_6mm -> MAPusart:OSHW_6mm
- moved Z5 3.30 mm to (120.8, 33.9)
- moved R4 1.00 mm to (122.0, 36.8)
- moved Z3 0.50 mm to (117.5, 44.5)
Connections:
- J3 pad 2: /D- -> /D-IN
- J3 pad 3: /D+ -> /D+IN
Routing:
- net /5V: track 21.9 -> 33.2 mm, vias 1 -> 2
- net /GND_U: track 63.3 -> 73.8 mm
- net /D-IN: track 0.00 -> 5.49 mm, vias 0 -> 1
- net /D+IN: track 0.00 -> 4.29 mm, vias 0 -> 1
- net /D+: track 17.6 -> 21.3 mm, vias 2 -> 1
- net /D-: track 16.3 -> 17.2 mm, vias 2 -> 1

Commit message: MAPusart complete and ready for prototyping
Parts:
- C10, C9: footprint MAPone.pretty:C_0805_HandSoldering -> MAPusart.pretty:C_0805_HandSoldering
- D4: footprint MAPone.pretty:LED-0805 -> MAPusart.pretty:LED-0805
- H10: footprint MAPone.pretty:Socket_Strip_Angled_1x06 -> MAPusart.pretty:Socket_Strip_Angled_1x06
- J3: footprint MAPone.pretty:USB_B_Micro -> MAPusart.pretty:USB_B_Micro
- R4: footprint MAPone.pretty:R_0805_HandSoldering -> MAPusart.pretty:R_0805_HandSoldering
- U3: footprint MAPone.pretty:qfn-28 -> MAPusart.pretty:qfn-28
- Z5: footprint MAPusart:OSHW_6mm -> MAPusart.pretty:OSHW_6mm
Changed lines of the file:
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@@
-(kicad_pcb (version 4) (host pcbnew 0.201411181401+5290~19~ubuntu14.10.1-product)
+(kicad_pcb (version 4) (host pcbnew "(2014-12-01 BZR 5309)-product")
   (general
     (links 32)
@@
   (page A4)
   (title_block
-    (title "MAPone - Bare Bones Arduino")
+    (title "MAPusart - USB to USART Bridge using CP2012")
     (rev v1)
     (company "Maker's Asylum : www.github.com/MakersAsylumIndia")
@@
       (drillshape 0)
       (scaleselection 1)
-      (outputdirectory /home/samata/projects-git/MAPusart/kicad/gerber/))
+      (outputdirectory /home/anool/projects-git/MAPusart/kicad/gerber/))
   )
   (net 0 "")
@@
     (uvia_drill 0.127)
   )
-  (module MAPone.pretty:C_0805_HandSoldering (layer F.Cu)
+  (module MAPusart.pretty:C_0805_HandSoldering (layer F.Cu)
     (at 121.925 42.75 90)
     (descr "Capacitor SMD 0805, hand soldering")
@@
     (pad 2 smd rect (at 1.25 0 90) (size 1.5 1.25) (layers F.Cu F.Paste F.Mask)
       (net 3 /GND_U))
-    (model /home/anool/projects-git/MAPone/kicad/MAPone_3D/C_0805N.wrl
+    (model /home/anool/projects-git/MAPusart/kicad/MAPusart_3D/C_0805N.wrl
       (at (xyz 0 0 0))
       (scale (xyz 1 1 1))
@@
     )
   )
-  (module MAPone.pretty:C_0805_HandSoldering (layer F.Cu)
+  (module MAPusart.pretty:C_0805_HandSoldering (layer F.Cu)
     (at 123.925 45.6 90)
     (descr "Capacitor SMD 0805, hand soldering")
@@
     (pad 2 smd rect (at 1.25 0 90) (size 1.5 1.25) (layers F.Cu F.Paste F.Mask)
       (net 3 /GND_U))
-    (model /home/anool/projects-git/MAPone/kicad/MAPone_3D/C_0805N.wrl
+    (model /home/anool/projects-git/MAPusart/kicad/MAPusart_3D/C_0805N.wrl
       (at (xyz 0 0 0))
       (scale (xyz 1 1 1))
@@
     )
   )
-  (module MAPone.pretty:USB_B_Micro (layer F.Cu)
+  (module MAPusart.pretty:USB_B_Micro (layer F.Cu)
     (at 117.5 34.25 270)
     (attr smd)
@@
     (pad T6 thru_hole circle (at -2.667 3.302 270) (size 1.905 1.905) (drill 1.27) (layers *.Cu *.Paste *.Mask F.SilkS)
       (net 3 /GND_U) (clearance 0.2032))
-    (model /home/anool/projects-git/MAPone/kicad/MAPone_3D/usb_B_micro_smd.wrl
+    (model /home/anool/projects-git/MAPusart/kicad/MAPusart_3D/usb_B_micro_smd.wrl
       (at (xyz -0.1 0 0))
       (scale (xyz 1 1 1))
@@
     )
   )
-  (module MAPone.pretty:R_0805_HandSoldering (layer F.Cu)
+  (module MAPusart.pretty:R_0805_HandSoldering (layer F.Cu)
     (at 122 36.8)
     (descr "Resistor SMD 0805, hand soldering")
@@
     (pad 2 smd rect (at 1.35 0) (size 1.5 1.3) (layers F.Cu F.Paste F.Mask)
       (net 1 "Net-(D4-Pad1)"))
-    (model /home/anool/projects-git/MAPone/kicad/MAPone_3D/R_0805.wrl
+    (model /home/anool/projects-git/MAPusart/kicad/MAPusart_3D/R_0805.wrl
       (at (xyz 0 0 0))
       (scale (xyz 1 1 1))
@@
     )
   )
-  (module MAPone.pretty:qfn-28 (layer F.Cu)
+  (module MAPusart.pretty:qfn-28 (layer F.Cu)
     (at 117.5 44)
     (descr "Plastic QFP, Microchip QFN-28")
@@
     (pad 7 smd rect (at 1.95072 2.84988) (size 0.35052 0.8001) (layers F.Cu F.Paste F.Mask)
       (net 2 /5V) (solder_mask_margin 0.07112) (clearance 0.1))
-    (model /home/anool/projects-git/MAPone/kicad/MAPone_3D/QFN28.wrl
+    (model /home/anool/projects-git/MAPusart/kicad/MAPusart_3D/QFN28.wrl
       (at (xyz 0 0 0))
       (scale (xyz 1 1 1))
@@
     )
   )
-  (module MAPone.pretty:LED-0805 (layer F.Cu)
+  (module MAPusart.pretty:LED-0805 (layer F.Cu)
     (at 123.4 33.1 90)
     (descr "LED 0805 smd package")
@@
     )
   )
-  (module MAPone.pretty:Socket_Strip_Angled_1x06 (layer B.Cu)
+  (module MAPusart.pretty:Socket_Strip_Angled_1x06 (layer B.Cu)
     (at 117.5 39)
     (descr "Through hole socket strip")
@@
     (pad 6 thru_hole circle (at -6.35 0) (size 1.524 1.524) (drill 1.016) (layers *.Cu *.Mask B.SilkS)
       (net 7 /RST))
-    (model projects-git/MAPone/kicad/MAPone_3D/Socket_Strip_Angled_1x06.wrl
+    (model projects-git/MAPusart/kicad/MAPusart_3D/Socket_Strip_Angled_1x06.wrl
       (at (xyz 0 0 0))
       (scale (xyz 1 1 1))
-      (rotate (xyz 0 0 0))
-    )
-  )
-  (module MAPusart.pretty:SOT-23-6 (layer B.Cu)
-    (at 114.7 35 270)
-    (fp_text reference D1 (at -2.1 -1.3 360) (layer B.SilkS)
-      (effects (font (size 0.8 0.8) (thickness 0.1)) (justify mirror))
-    )
-    (fp_text value USBLC6-2 (at 0.0635 0 270) (layer B.SilkS) hide
-      (effects (font (size 0.50038 0.50038) (thickness 0.0762)) (justify mirror))
-    )
-    (fp_line (start -0.508 -0.762) (end -1.27 -0.254) (layer B.SilkS) (width 0.15))
-    (fp_line (start 1.27 -0.762) (end -1.3335 -0.762) (layer B.SilkS) (width 0.15))
-    (fp_line (start -1.3335 -0.762) (end -1.3335 0.762) (layer B.SilkS) (width 0.15))
-    (fp_line (start -1.3335 0.762) (end 1.27 0.762) (layer B.SilkS) (width 0.15))
-    (fp_line (start 1.27 0.762) (end 1.27 -0.762) (layer B.SilkS) (width 0.15))
-    (pad 6 smd rect (at -0.9525 1.27 270) (size 0.70104 1.00076) (layers B.Cu B.Paste B.Mask)
-      (net 8 /D+))
-    (pad 5 smd rect (at 0 1.27 270) (size 0.70104 1.00076) (layers B.Cu B.Paste B.Mask)
-      (net 2 /5V))
-    (pad 4 smd rect (at 0.9525 1.27 270) (size 0.70104 1.00076) (layers B.Cu B.Paste B.Mask)
-      (net 9 /D-))
-    (pad 3 smd rect (at 0.9525 -1.27 270) (size 0.70104 1.00076) (layers B.Cu B.Paste B.Mask)
-      (net 10 /D-IN))
-    (pad 2 smd rect (at 0 -1.27 270) (size 0.70104 1.00076) (layers B.Cu B.Paste B.Mask)
-      (net 3 /GND_U))
-    (pad 1 smd rect (at -0.9525 -1.27 270) (size 0.70104 1.00076) (layers B.Cu B.Paste B.Mask)
-      (net 11 /D+IN))
-    (model smd/SOT23_6.wrl
-      (at (xyz 0 0 0))
-      (scale (xyz 0.11 0.11 0.11))
       (rotate (xyz 0 0 0))
     )
@@
       (xy -1.178278 0.308043) (xy -1.178278 0.308043)) (layer B.SilkS) (width 0.1))
   )
-  (module MAPusart:OSHW_6mm (layer B.Cu)
+  (module MAPusart.pretty:OSHW_6mm (layer B.Cu)
     (at 120.8 33.9 180)
     (fp_text reference Z5 (at 0 -3.54076 180) (layer B.SilkS) hide
@@
       (xy -2.02438 -2.99974)) (layer B.SilkS) (width 0.00254))
   )
+  (module MAPusart.pretty:SOT-23-6 (layer B.Cu)
+    (at 114.7 35 270)
+    (fp_text reference D1 (at -2.1 -1.3 360) (layer B.SilkS)
+      (effects (font (size 0.8 0.8) (thickness 0.1)) (justify mirror))
+    )
+    (fp_text value USBLC6-2 (at 0.0635 0 270) (layer B.SilkS) hide
+      (effects (font (size 0.50038 0.50038) (thickness 0.0762)) (justify mirror))
+    )
+    (fp_line (start -0.508 -0.762) (end -1.27 -0.254) (layer B.SilkS) (width 0.15))
+    (fp_line (start 1.27 -0.762) (end -1.3335 -0.762) (layer B.SilkS) (width 0.15))
+    (fp_line (start -1.3335 -0.762) (end -1.3335 0.762) (layer B.SilkS) (width 0.15))
+    (fp_line (start -1.3335 0.762) (end 1.27 0.762) (layer B.SilkS) (width 0.15))
+    (fp_line (start 1.27 0.762) (end 1.27 -0.762) (layer B.SilkS) (width 0.15))
+    (pad 6 smd rect (at -0.9525 1.27 270) (size 0.70104 1.00076) (layers B.Cu B.Paste B.Mask)
+      (net 8 /D+))
+    (pad 5 smd rect (at 0 1.27 270) (size 0.70104 1.00076) (layers B.Cu B.Paste B.Mask)
+      (net 2 /5V))
+    (pad 4 smd rect (at 0.9525 1.27 270) (size 0.70104 1.00076) (layers B.Cu B.Paste B.Mask)
+      (net 9 /D-))
+    (pad 3 smd rect (at 0.9525 -1.27 270) (size 0.70104 1.00076) (layers B.Cu B.Paste B.Mask)
+      (net 10 /D-IN))
+    (pad 2 smd rect (at 0 -1.27 270) (size 0.70104 1.00076) (layers B.Cu B.Paste B.Mask)
+      (net 3 /GND_U))
+    (pad 1 smd rect (at -0.9525 -1.27 270) (size 0.70104 1.00076) (layers B.Cu B.Paste B.Mask)
+      (net 11 /D+IN))
+    (model projects-git/MAPusart/kicad/MAPusart_3D/SOT23_6.wrl
+      (at (xyz 0 0 0))
+      (scale (xyz 0.11 0.11 0.11))
+      (rotate (xyz 0 0 0))
+    )
+  )
   (gr_line (start 110 32) (end 110 49) (angle 90) (layer Edge.Cuts) (width 0.1))
